File: easun-smw-dsp/easun-smw-dsp.kicad_sch (KiCad schematic)
At the start: 375 parts, among them CN1 (JTAG), CN11 Conn_01x16, CN2 (TO MPPT), CN5 (TO CAN), CN6 (TO COM), CN8 (TO LED), CN9 Conn_01x16, J10 Conn_01x16, Q3 MMBT2222A, Q5 MMBT2222A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

Commit message: Add files via upload
Connections:
- net CN11_PIN7 is gone; now on net CN11/7: U13.10 (O7)
- net DSP_PIN2: no longer CN11.15 (Pin_15), R93.2
- net SFT_RELAY renamed GRID_L_RELAY
- new net DSP_PIN1: CN11.15 (Pin_15), R93.2
Other:
- moved on the sheet: Q6, R196, R197, R198
