File: easun-smw-scr/easun-smw-scr.kicad_sch (KiCad schematic)
At the start: 71 parts, among them CN1 Conn_01x08, CN2 BDM, Q1 TYN8012, Q2 TYN8012, Q3 TYN8012, Q4 TYN8012, Q5 B095N, Q6 B095N, Q7 BTNT2, U1 MC9S08FL8CLC

Commit message: Add files via upload
Connections:
- net GRID_N_REQ: now reaches CN1.7 (Pin_7), U1.26 (PTA0)
Other:
- note added: "SCR_GRID"
- note added: "SCR_OP"
Changed lines of the file:
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@@
 		(comment 1 "Board no. 16-501418-01G")
 	)
+	(text "SCR_GRID"
+		(exclude_from_sim no)
+		(at 279.4 52.07 90)
+		(effects
+			(font
+				(size 1.27 1.27)
+			)
+		)
+	)
+	(text "SCR_OP"
+		(exclude_from_sim no)
+		(at 279.4 124.46 90)
+		(effects
+			(font
+				(size 1.27 1.27)
+			)
+		)
+	)
 	(junction
 		(at 250.19 114.3)
@@
 		(effects
 			(font
+				(size 1.27 1.27)
+			)
+			(justify left bottom)
+		)
+	)
+	(label "GRID_N_REQ"
+		(at 26.67 105.41 0)
+		(effects
+			(font
